File: hardware/SensorBoard.sch (EAGLE design)
At the start: 222 parts, among them IC1 SI7006-A10-IM, IC3 DWM1000, IC4 BMP280, IC5 FT232R, Q1 MC-306, T3 BC337, T4 BC337, U1 ESP-WROOM-32, U3 UM18533, X2 SMA-142-0711-821/826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

Commit message: Cleaned hardware data.
Parts:
- removed JP30, JP31, JP33, JP34, JP35: (no value), pinhead:PINHD-1X1
- added JPGND, JPGND1, JPGND2, JPVCC, JPVCC1: (no value), pinhead:PINHD-1X1
Connections:
- net +3V3: now also JPVCC.1, JPVCC1.1; no longer JP30.1, JP34.1
- net GND: now also JPGND.1, JPGND1.1, JPGND2.1; no longer JP31.1, JP33.1, JP35.1
Other:
- note added: "Bedrich Said"
- note added: "Diploma Thesis Faculty of Informatics Masaryk university, Brno In cooperation with: Robotarna (RobotikaBrno.cz)"
- note added: "v1.0"
- note removed: "RobotikaBrno"
- note removed: "RobotikaBrno.cz Robotarna"
- note removed: "github:roboticsbrno/ RB3200-ESP32universal RobotikaBrno.cz Robotarna CC BY-SA 4.0"
- note removed: "v3.1"
